File: CEI-TOOL.kicad_pcb (KiCad board)
At the start: 2 copper layers, 71.5 x 33 mm, 61 parts, among them J1 TYPE-C-31-M-12, J2 532610871, J3 S2B-PH-SM4-TB_LF__SN_, J4 SM04B-SRSS-TB, J6 SM02B-SRSS-TB_LF__SN_, U1 ESP32-C3-MINI-1, U2 XC6220B331PR-G, U3 BQ24075RGTT, U4 USBLC6-2SC6

Commit message: edit
Parts:
- removed D1: SMBJ5.0A, SMBJ5.0A:DIOM4336X265N
- removed J3: S2B-PH-SM4-TB_LF__SN_, S2B-PH-SM4-TB_LF__SN_:JST_S2B-PH-SM4-TB_LF__SN_
- removed TP8: TestPoint_Pad_D1.0mm, TestPoint:TestPoint_Pad_D1.0mm
- added C14: 22µF, Capacitor_SMD:C_0603_1608Metric, F.Cu at (146.7, 107.0)
- added D4: SMF5.0A, SMF5.0A:P37_SOD-123FL, F.Cu at (169.4, 102.0)
- added J5: 532610271, 532610271:MOLEX_532610271, F.Cu at (181.5, 102.5)
- added R22: 10kΩ, Resistor_SMD:R_0603_1608Metric, F.Cu at (130.5, 91.5)
- C8: value 0.1µF -> 1µF
- R10, R8: value 4.7kΩ -> 2.2kΩ
- turned D3 to 180 degrees
- renumbered BOOT to EN
Connections:
- U1 pad 22: TP-GPIO8 -> Net-(U1-GPIO8)
Routing:
- net +3.3V: track 256.6 -> 286.2 mm
- net Net-(U1-GPIO8): track 0.00 -> 5.15 mm
- net TP-GPIO8: track 4.47 -> 0.00 mm
- net BAT: track 32.0 -> 29.1 mm
- net BOOT_BTN: track 24.0 -> 22.1 mm
- net TP-VBUS: track 30.5 -> 31.6 mm
- net GND: vias 118 -> 114

Commit message: 회소 수정
Connections:
- U1 pad 16: USB_PGOOD -> SPI_CS
- U1 pad 19: SPI_CS -> USB_PGOOD
Routing:
- net SPI_CS: track 28.1 -> 32.4 mm, vias 0 -> 2
- net USB_PGOOD: track 49.7 -> 52.2 mm
- net GND: track 30.6 -> 29.9 mm, vias 114 -> 113
