File: CEI-TOOL.kicad_sch (KiCad schematic)
At the start: 49 parts, among them J1 TYPE-C-31-M-12, J2 532610871, J3 S2B-PH-SM4-TB_LF__SN_, J4 SM04B-SRSS-TB, J6 SM02B-SRSS-TB_LF__SN_, U1 ESP32-C3-MINI-1, U2 XC6220B331PR-G, U3 BQ24075RGTT, U4 USBLC6-2SC6

Commit message: edit
Parts:
- removed D1: SMBJ5.0A, SMBJ5.0A:DIOM4336X265N, symbol SMBJ5.0A:SMBJ5.0A
- removed J3: S2B-PH-SM4-TB_LF__SN_, S2B-PH-SM4-TB_LF__SN_:JST_S2B-PH-SM4-TB_LF__SN_, symbol S2B-PH-SM4-TB_LF__SN_:S2B-PH-SM4-TB_LF__SN_
- added C14: 22µF, Capacitor_SMD:C_0603_1608Metric, symbol Device:C
- added D4: SMF5.0A, SMF5.0A:P37_SOD-123FL, symbol SMF5.0A:SMF5.0A
- added J5: 532610271, 532610271:MOLEX_532610271, symbol 532610271:532610271
- added R22: 10kΩ, Resistor_SMD:R_0603_1608Metric, symbol Device:R
- C8: value 0.1µF -> 1µF
- R10, R8: value 4.7kΩ -> 2.2kΩ
Connections:
- net +3.3V: now also R22.2
- net BAT: now also J5.1
- net GND: now also C14.2, D4.2 (A), J5.2, J5.S1 (SHIELD1), J5.S2 (SHIELD2)
- net VBUS: now also D4.1 (C)
- net VSYS: now also C14.1
- net TP-GPIO8: no longer names the net of U1.22 (GPIO8)
- net TP-GPIO8: now also R22.1
Other:
- moved on the sheet: C11, C4, C5, R1, R13, R15, R2, S3, U2

Commit message: 회소 수정
Connections:
- net SPI_CS: now also U1.16 (GPIO10); no longer U1.19 (GPIO5/ADC2_CH0)
- net USB_PGOOD: now also U1.19 (GPIO5/ADC2_CH0); no longer U1.16 (GPIO10)
Changed lines of the file:
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@@
 	(wire
 		(pts
-			(xy 266.7 172.72) (xy 261.62 172.72)
+			(xy 266.7 172.72) (xy 262.89 172.72)
 		)
 		(stroke
@@
 	(wire
 		(pts
-			(xy 271.78 172.72) (xy 274.32 172.72)
+			(xy 271.78 184.15) (xy 278.13 184.15)
 		)
 		(stroke
@@
 	(wire
 		(pts
-			(xy 294.64 182.88) (xy 294.64 184.15)
+			(xy 290.83 184.15) (xy 290.83 185.42)
 		)
 		(stroke
@@
 	(wire
 		(pts
-			(xy 274.32 184.15) (xy 278.13 184.15)
-		)
-		(stroke
-			(width 0)
-			(type default)
-		)
-	)
-	(wire
-		(pts
 			(xy 278.13 152.4) (xy 266.7 152.4)
 		)
@@
 	(wire
 		(pts
-			(xy 274.32 167.64) (xy 276.86 167.64)
+			(xy 274.32 171.45) (xy 276.86 171.45)
 		)
 		(stroke
@@
 	(wire
 		(pts
-			(xy 261.62 172.72) (xy 261.62 175.26)
+			(xy 262.89 172.72) (xy 262.89 177.8)
 		)
 		(stroke
@@
 	(wire
 		(pts
-			(xy 273.05 171.45) (xy 276.86 171.45)
+			(xy 273.05 176.53) (xy 276.86 176.53)
 		)
 		(stroke
@@
 	(wire
 		(pts
-			(xy 271.78 160.02) (xy 271.78 172.72)
+			(xy 271.78 160.02) (xy 271.78 184.15)
 		)
 		(stroke
@@
 	(wire
 		(pts
-			(xy 294.64 184.15) (xy 285.75 184.15)
+			(xy 290.83 184.15) (xy 285.75 184.15)
 		)
 		(stroke
@@
 	(wire
 		(pts
-			(xy 273.05 157.48) (xy 273.05 171.45)
+			(xy 273.05 157.48) (xy 273.05 176.53)
 		)
 		(stroke
@@
 	(wire
 		(pts
-			(xy 274.32 172.72) (xy 274.32 184.15)
-		)
-		(stroke
-			(width 0)
-			(type default)
-		)
-	)
-	(wire
-		(pts
 			(xy 330.2 139.7) (xy 334.01 139.7)
 		)
@@
 	(wire
 		(pts
-			(xy 318.77 72.39) (xy 316.23 72.39)
+			(xy 318.77 72.39) (xy 314.96 72.39)
 		)
 		(stroke
@@
 	(wire
 		(pts
-			(xy 274.32 154.94) (xy 274.32 167.64)
+			(xy 274.32 154.94) (xy 274.32 171.45)
 		)
 		(stroke
@@
 		)
 	)
+	(global_label "SPI_CS"
+		(shape input)
+		(at 262.89 177.8 270)
+		(fields_autoplaced yes)
+		(effects
+			(font
+				(size 1.27 1.27)
+			)
+			(justify right)
+		)
+		(property "Intersheetrefs" "${INTERSHEET_REFS}"
+			(at 262.89 187.3166 90)
+			(effects
+				(font
+					(size 1.27 1.27)
+				)
+				(justify right)
+				(hide yes)
+			)
+		)
+	)
 	(global_label "USB_D-"
 		(shape input)
@@
 		)
 	)
+	(global_label "USB_PGOOD"
+		(shape input)
+		(at 278.13 153.67 270)
+		(fields_autoplaced yes)
+		(effects
+			(font
+				(size 1.27 1.27)
+			)
+			(justify right)
+		)
+		(property "Intersheetrefs" "${INTERSHEET_REFS}"
+			(at 278.13 167.9038 90)
+			(effects
+				(font
+					(size 1.27 1.27)
+				)
+				(justify right)
+				(hide yes)
+			)
+		)
+	)
 	(global_label "SPI_DC"
 		(shape input)
@@
 		)
 	)
-	(global_label "SPI_CS"
-		(shape input)
-		(at 278.13 153.67 270)
-		(fields_autoplaced yes)
-		(effects
-			(font
-				(size 1.27 1.27)
-			)
-			(justify right)
-		)
-		(property "Intersheetrefs" "${INTERSHEET_REFS}"
-			(at 278.13 163.1866 90)
-			(effects
-				(font
-					(size 1.27 1.27)
-				)
-				(justify right)
-				(hide yes)
-			)
-		)
-	)
 	(global_label "SPI_DC"
 		(shape input)
@@
 		)
 	)
-	(global_label "USB_PGOOD"
-		(shape input)
-		(at 261.62 175.26 270)
-		(fields_autoplaced yes)
-		(effects
-			(font
-				(size 1.27 1.27)
-			)
-			(justify right)
-		)
-		(property "Intersheetrefs" "${INTERSHEET_REFS}"
-			(at 261.62 189.4938 90)
-			(effects
-				(font
-					(size 1.27 1.27)
-				)
-				(justify right)
-				(hide yes)
-			)
-		)
-	)
 	(global_label "SPI_CLK"
 		(shape input)
-		(at 276.86 167.64 0)
+		(at 276.86 171.45 0)
 		(fields_autoplaced yes)
 		(effects
@@
 		)
 		(property "Intersheetrefs" "${INTERSHEET_REFS}"
-			(at 287.4652 167.64 0)
+			(at 287.4652 171.45 0)
 			(effects
 				(font
@@
 	(global_label "SPI_MOSI(DIN)"
 		(shape input)
-		(at 276.86 171.45 0)
+		(at 276.86 176.53 0)
 		(fields_autoplaced yes)
 		(effects
@@
 		)
 		(property "Intersheetrefs" "${INTERSHEET_REFS}"
-			(at 293.392 171.45 0)
+			(at 293.392 176.53 0)
 			(effects
 				(font
@@
 	(global_label "SPI_CS"
 		(shape input)
-		(at 316.23 72.39 180)
+		(at 314.96 72.39 180)
 		(fields_autoplaced yes)
 		(effects
@@
 		)
 		(property "Intersheetrefs" "${INTERSHEET_REFS}"
-			(at 306.7134 72.39 0)
+			(at 305.4434 72.39 0)
 			(effects
 				(font
@@
 	(symbol
 		(lib_id "power:+3.3V")
-		(at 294.64 182.88 0)
+		(at 290.83 185.42 180)
 		(unit 1)
 		(exclude_from_sim no)
@@
 		(dnp no)
 		(property "Reference" "#PWR037"
-			(at 294.64 186.69 0)
+			(at 290.83 181.61 0)
 			(effects
 				(font
@@
 		)
 		(property "Value" "+3.3V"
-			(at 294.64 177.8 0)
+			(at 290.83 190.5 0)
 			(effects
 				(font
@@
 		)
 		(property "Footprint" ""
-			(at 294.64 182.88 0)
+			(at 290.83 185.42 0)
 			(effects
 				(font
@@
 		)
 		(property "Datasheet" ""
-			(at 294.64 182.88 0)
+			(at 290.83 185.42 0)
 			(effects
 				(font
@@
 		)
 		(property "Description" "Power symbol creates a global label with name \"+3.3V\""
-			(at 294.64 182.88 0)
+			(at 290.83 185.42 0)
 			(effects
 				(font
